Commit message: Updated base STL, added Soumith's actuators and aligned all

File: src/whac-a-mole_description/urdf/whac-a-mole.urdf (robot description, URDF)
Before this commit: robot whac-a-mole, 6 links, 5 joints
Links:
- added link slider_link_1, mass 0.5; collision cylinder length=1.00 radius=0.2; visual cylinder length=1.00 radius=0.2
- added link slider_link_2, mass 0.5; collision cylinder length=1.00 radius=0.2; visual cylinder length=1.00 radius=0.2
- added link slider_link_3, mass 0.5; collision cylinder length=1.00 radius=0.2; visual cylinder length=1.00 radius=0.2
- added link slider_link_4, mass 0.5; collision cylinder length=1.00 radius=0.2; visual cylinder length=1.00 radius=0.2
- link linear_actuator_1: mass 0.5 -> 1.0; geometry collision box size=1 1 0.5; visual box size=1 1 0.5
- link linear_actuator_2: mass 0.5 -> 1.0; geometry collision box size=1 1 0.5; visual box size=1 1 0.5
- link linear_actuator_3: mass 0.5 -> 1.0; geometry collision box size=1 1 0.5; visual box size=1 1 0.5
- link linear_actuator_4: mass 0.5 -> 1.0; geometry collision box size=1 1 0.5; visual box size=1 1 0.5
Joints:
- added joint slider_joint_1: type prismatic, parent linear_actuator_1, child slider_link_1, origin xyz=0 0 0 rpy=0 0 0, axis 0 0 1, limit lower=0.0 upper=0.3 effort=100.0 velocity=1.0
- added joint slider_joint_2: type prismatic, parent linear_actuator_2, child slider_link_2, origin xyz=0 0 0 rpy=0 0 0, axis 0 0 1, limit lower=0.0 upper=0.3 effort=100.0 velocity=1.0
- added joint slider_joint_3: type prismatic, parent linear_actuator_3, child slider_link_3, origin xyz=0 0 0 rpy=0 0 0, axis 0 0 1, limit lower=0.0 upper=0.3 effort=100.0 velocity=1.0
- added joint slider_joint_4: type prismatic, parent linear_actuator_4, child slider_link_4, origin xyz=0 0 0 rpy=0 0 0, axis 0 0 1, limit lower=0.0 upper=0.3 effort=100.0 velocity=1.0
- joint base_to_linear_actuator_1: origin xyz=0.1 0 0 rpy=0 0 0 -> xyz=-1 -8 3 rpy=0 0 0
- joint base_to_linear_actuator_2: origin xyz=15 0 0 rpy=0 0 0 -> xyz=-3 -8 3 rpy=0 0 0
- joint base_to_linear_actuator_3: origin xyz=30 0 0 rpy=0 0 0 -> xyz=-7 -8 3 rpy=0 0 0
- joint base_to_linear_actuator_4: origin xyz=45 0 0 rpy=0 0 0 -> xyz=-9 -8 3 rpy=0 0 0
- joint world_joint: origin xyz=2 0 1.5 rpy=0 0 0 -> xyz=5.5 4 0 rpy=0 0 0

Commit message: Moving linear actuators! Added basic code

File: src/whac-a-mole_description/urdf/whac-a-mole.urdf (robot description, URDF)
Before this commit: robot whac-a-mole, 10 links, 9 joints
Links:
- link base: geometry visual mesh filename=package://whac-a-mole_description/meshes/Base.stl
- link linear_actuator_1: geometry visual box size=1 1 0.5
- link linear_actuator_2: geometry visual box size=1 1 0.5
- link linear_actuator_3: geometry visual box size=1 1 0.5
- link linear_actuator_4: geometry visual box size=1 1 0.5
- link slider_link_1: geometry visual cylinder length=1.00 radius=0.2
- link slider_link_2: geometry visual cylinder length=1.00 radius=0.2
- link slider_link_3: geometry visual cylinder length=1.00 radius=0.2
- link slider_link_4: geometry visual cylinder length=1.00 radius=0.2
Joints:
- joint base_to_linear_actuator_1: origin xyz=-1 -8 3 rpy=0 0 0 -> xyz=4 -4 3 rpy=0 0 0; parent base -> world
- joint base_to_linear_actuator_2: origin xyz=-3 -8 3 rpy=0 0 0 -> xyz=2 -4 3 rpy=0 0 0; parent base -> world
- joint base_to_linear_actuator_3: origin xyz=-7 -8 3 rpy=0 0 0 -> xyz=-1 -4 3 rpy=0 0 0; parent base -> world
- joint base_to_linear_actuator_4: origin xyz=-9 -8 3 rpy=0 0 0 -> xyz=-3 -4 3 rpy=0 0 0; parent base -> world
- joint slider_joint_1: origin xyz=0 0 0 rpy=0 0 0 -> xyz=0 0 0.75 rpy=0 0 0
- joint slider_joint_2: origin xyz=0 0 0 rpy=0 0 0 -> xyz=0 0 0.75 rpy=0 0 0
- joint slider_joint_3: origin xyz=0 0 0 rpy=0 0 0 -> xyz=0 0 0.75 rpy=0 0 0
- joint slider_joint_4: origin xyz=0 0 0 rpy=0 0 0 -> xyz=0 0 0.75 rpy=0 0 0

Commit message: Refactor actuator movement logic to use sine wave for smoother transitions and update URDF to reflect new actuator dimensions and joint configurations.

File: src/whac-a-mole_description/urdf/whac-a-mole.urdf (robot description, URDF)
Before this commit: robot whac-a-mole, 10 links, 9 joints
Links:
- link slider_link_1: geometry visual cylinder length=3.00 radius=0.2
- link slider_link_2: geometry visual cylinder length=3.00 radius=0.2
- link slider_link_3: geometry visual cylinder length=3.00 radius=0.2
- link slider_link_4: geometry visual cylinder length=3.00 radius=0.2
Joints:
- removed joint base_to_linear_actuator_1
- removed joint base_to_linear_actuator_2
- removed joint base_to_linear_actuator_3
- removed joint base_to_linear_actuator_4
- added joint base_to_slider_link_1: type fixed, parent slider_link_1, child linear_actuator_1, origin xyz=0 0 -1.75 rpy=0 0 0
- added joint base_to_slider_link_2: type fixed, parent slider_link_2, child linear_actuator_2, origin xyz=0 0 -1.75 rpy=0 0 0
- added joint base_to_slider_link_3: type fixed, parent slider_link_3, child linear_actuator_3, origin xyz=0 0 -1.75 rpy=0 0 0
- added joint base_to_slider_link_4: type fixed, parent slider_link_4, child linear_actuator_4, origin xyz=0 0 -1.75 rpy=0 0 0
- joint slider_joint_1: limit lower=0.0 upper=0.3 effort=100.0 velocity=1.0 -> lower=-2.25 upper=0.4 effort=100.0 velocity=1.0; origin xyz=0 0 0.75 rpy=0 0 0 -> xyz=4 -4 4.75 rpy=0 0 0; parent linear_actuator_1 -> world
- joint slider_joint_2: limit lower=0.0 upper=0.3 effort=100.0 velocity=1.0 -> lower=-2.25 upper=0.4 effort=100.0 velocity=1.0; origin xyz=0 0 0.75 rpy=0 0 0 -> xyz=2 -4 4.75 rpy=0 0 0; parent linear_actuator_2 -> world
- joint slider_joint_3: limit lower=0.0 upper=0.3 effort=100.0 velocity=1.0 -> lower=-2.25 upper=0.4 effort=100.0 velocity=1.0; origin xyz=0 0 0.75 rpy=0 0 0 -> xyz=-1 -4 4.75 rpy=0 0 0; parent linear_actuator_3 -> world
- joint slider_joint_4: limit lower=0.0 upper=0.3 effort=100.0 velocity=1.0 -> lower=-2.25 upper=0.4 effort=100.0 velocity=1.0; origin xyz=0 0 0.75 rpy=0 0 0 -> xyz=-3 -4 4.75 rpy=0 0 0; parent linear_actuator_4 -> world

Commit message: Add button mechanisms and update URDF for new prismatic joints and spring effects

File: src/whac-a-mole_description/urdf/whac-a-mole.urdf (robot description, URDF)
Before this commit: robot whac-a-mole, 10 links, 9 joints
Links:
- added link button_base_1, mass 0.1; visual box size=1 1 1
- added link button_base_2, mass 0.1; visual box size=1 1 1
- added link button_base_3, mass 0.1; visual box size=1 1 1
- added link button_base_4, mass 0.1; visual box size=1 1 1
- added link button_top_1, mass 0.1; collision cylinder length=0.3 radius=0.45; visual cylinder length=0.3 radius=0.45
- added link button_top_2, mass 0.1; collision cylinder length=0.3 radius=0.45; visual cylinder length=0.3 radius=0.45
- added link button_top_3, mass 0.1; collision cylinder length=0.3 radius=0.45; visual cylinder length=0.3 radius=0.45
- added link button_top_4, mass 0.1; collision cylinder length=0.3 radius=0.45; visual cylinder length=0.3 radius=0.45
- link linear_actuator_1: geometry collision box size=1 1 0.5; visual box size=1 1 0.5
- link linear_actuator_2: geometry collision box size=1 1 0.5; visual box size=1 1 0.5
- link linear_actuator_3: geometry collision box size=1 1 0.5; visual box size=1 1 0.5
- link linear_actuator_4: geometry collision box size=1 1 0.5; visual box size=1 1 0.5
Joints:
- added joint button_1_base_to_world: type fixed, parent world, child button_base_1, origin xyz=4 -4 0.5 rpy=0 0 0
- added joint button_2_base_to_world: type fixed, parent world, child button_base_2, origin xyz=2 -4 0.5 rpy=0 0 0
- added joint button_3_base_to_world: type fixed, parent world, child button_base_3, origin xyz=-1 -4 0.5 rpy=0 0 0
- added joint button_4_base_to_world: type fixed, parent world, child button_base_4, origin xyz=-3 -4 0.5 rpy=0 0 0
- added joint button_joint_1: type prismatic, parent button_base_1, child button_top_1, origin xyz=0 0 1.65 rpy=0 0 0, axis 0 0 1, limit lower=-1 upper=0 effort=10 velocity=0.1
- added joint button_joint_2: type prismatic, parent button_base_2, child button_top_2, origin xyz=0 0 1.65 rpy=0 0 0, axis 0 0 1, limit lower=-1 upper=0 effort=10 velocity=0.1
- added joint button_joint_3: type prismatic, parent button_base_3, child button_top_3, origin xyz=0 0 1.65 rpy=0 0 0, axis 0 0 1, limit lower=-1 upper=0 effort=10 velocity=0.1
- added joint button_joint_4: type prismatic, parent button_base_4, child button_top_4, origin xyz=0 0 1.65 rpy=0 0 0, axis 0 0 1, limit lower=-1 upper=0 effort=10 velocity=0.1

Commit message: Add button joint controllers and update actuator movement logic (sine wave button presses)

File: src/whac-a-mole_description/urdf/whac-a-mole.urdf (robot description, URDF)
Before this commit: robot whac-a-mole, 18 links, 17 joints
Joints:
- joint button_joint_1: limit lower=-1 upper=0 effort=10 velocity=0.1 -> lower=-0.5 upper=0 effort=10 velocity=0.1; origin xyz=0 0 1.65 rpy=0 0 0 -> xyz=0 0 0.65 rpy=0 0 0
- joint button_joint_2: limit lower=-1 upper=0 effort=10 velocity=0.1 -> lower=-0.5 upper=0 effort=10 velocity=0.1; origin xyz=0 0 1.65 rpy=0 0 0 -> xyz=0 0 0.65 rpy=0 0 0
- joint button_joint_3: limit lower=-1 upper=0 effort=10 velocity=0.1 -> lower=-0.5 upper=0 effort=10 velocity=0.1; origin xyz=0 0 1.65 rpy=0 0 0 -> xyz=0 0 0.65 rpy=0 0 0
- joint button_joint_4: limit lower=-1 upper=0 effort=10 velocity=0.1 -> lower=-0.5 upper=0 effort=10 velocity=0.1; origin xyz=0 0 1.65 rpy=0 0 0 -> xyz=0 0 0.65 rpy=0 0 0

Commit message: Enhance user input handling and adjust button/hammer positions in whac-a-mole game

File: src/whac-a-mole_description/urdf/whac-a-mole.urdf (robot description, URDF)
Before this commit: robot whac-a-mole, 18 links, 17 joints
Joints:
- joint button_1_base_to_world: origin xyz=4 -4 0.5 rpy=0 0 0 -> xyz=-3 -4 0.5 rpy=0 0 0
- joint button_2_base_to_world: origin xyz=2 -4 0.5 rpy=0 0 0 -> xyz=-1 -4 0.5 rpy=0 0 0
- joint button_3_base_to_world: origin xyz=-1 -4 0.5 rpy=0 0 0 -> xyz=2 -4 0.5 rpy=0 0 0
- joint button_4_base_to_world: origin xyz=-3 -4 0.5 rpy=0 0 0 -> xyz=4 -4 0.5 rpy=0 0 0
- joint slider_joint_1: origin xyz=4 -4 4.75 rpy=0 0 0 -> xyz=-3 -4 4.75 rpy=0 0 0
- joint slider_joint_2: origin xyz=2 -4 4.75 rpy=0 0 0 -> xyz=-1 -4 4.75 rpy=0 0 0
- joint slider_joint_3: origin xyz=-1 -4 4.75 rpy=0 0 0 -> xyz=2 -4 4.75 rpy=0 0 0
- joint slider_joint_4: origin xyz=-3 -4 4.75 rpy=0 0 0 -> xyz=4 -4 4.75 rpy=0 0 0
